File: vocorebreakout/vocorebreakout.kicad_sch (KiCad schematic)
At the start: 53 parts, among them J1 8P8C_LED_Shielded, J10 Top, J11 Right, J12 Conn_02x04_Odd_Even, J2 8P8C_LED_Shielded, J3 8P8C_LED_Shielded, J4 Conn_01x03, J5 Left, J6 Bottom, J7 Conn_02x04_Top_Bottom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

Commit message: vocorebreakout: Move SPI flash to bottom and ethernet port to #2
Connections:
- net RD2+: now also J5.11 (Pin_11); no longer J5.15 (Pin_15)
- net RD2-: now also J5.12 (Pin_12); no longer J5.16 (Pin_16)
- net TD2+: now also J5.13 (Pin_13); no longer J6.2 (Pin_2)
- net TD2-: now also J5.14 (Pin_14); no longer J6.3 (Pin_3)
Changed lines of the file:
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@@
     (effects (font (size 1.27 1.27)) (justify right bottom))
   )
-  (label "TD2-" (at 69.85 129.54 180)
-    (effects (font (size 1.27 1.27)) (justify right bottom))
+  (label "TD2-" (at 82.55 114.3 0)
+    (effects (font (size 1.27 1.27)) (justify left bottom))
   )
   (label "ROUT" (at 86.36 21.59 0)
@@
     (effects (font (size 1.27 1.27)) (justify left bottom))
   )
-  (label "RD2+" (at 69.85 116.84 180)
+  (label "RD2+" (at 69.85 111.76 180)
     (effects (font (size 1.27 1.27)) (justify right bottom))
   )
@@
     (effects (font (size 1.27 1.27)) (justify right bottom))
   )
-  (label "TD2+" (at 82.55 127 0)
-    (effects (font (size 1.27 1.27)) (justify left bottom))
+  (label "TD2+" (at 69.85 114.3 180)
+    (effects (font (size 1.27 1.27)) (justify right bottom))
   )
   (label "HOST_SDA" (at 158.75 180.34 0)
@@
     (effects (font (size 1.27 1.27)) (justify right bottom))
   )
-  (label "RD2-" (at 82.55 116.84 0)
+  (label "RD2-" (at 82.55 111.76 0)
     (effects (font (size 1.27 1.27)) (justify left bottom))
   )
